File: boards/RP2350A_chip_board/RP2350A_chip_board.kicad_sch (KiCad schematic)
At the start: 39 parts, among them J1 Conn_01x02, J2 Conn_01x03, J3 Conn_01x16, J4 Conn_01x03, J5 Conn_01x01, J6 Conn_01x01, U1 W25Q128JVS, U2 RP2350_60QFN, Y1 ABM8-272-T3

Commit message: Add Broker board
Parts:
- C12, C13: footprint RP2350_60QFN_minimal:C_0402_1005Metric_small_pads -> RP2350A_chip_board:C_0402_1005Metric_small_pads
- L1: footprint RP2350_60QFN_minimal:L_pol_2016 -> RP2350A_chip_board:L_pol_2016
- U1: symbol RP2350_60QFN_minimal-rescue:W25Q128JVS-Memory_Flash -> RP2350A_chip_board-rescue:W25Q128JVS-Memory_Flash
- U2: footprint RP2350_60QFN_minimal:RP2350-QFN-60-1EP_7x7_P0.4mm_EP3.4x3.4mm_ThermalVias -> RP2350A_chip_board:RP2350-QFN-60-1EP_7x7_P0.4mm_EP3.4x3.4mm_ThermalVias
