File: boards/RP2350B_chip_board/RP2350B_chip_board.kicad_sch (KiCad schematic)
At the start: 49 parts, among them J1 USB_B_Micro, J2 Conn_02x26_Odd_Even, J3 Conn_02x26_Odd_Even, J4 SM03B-SRSS-TB, SW1 SW_Push, SW2 SW_Push, U1 RP2350_80QFN, U2 NCP1117-3.3_SOT223, U3 W25Q128JVS, U4 DNF, Y1 ABM8-272-T3

Commit message: Add Broker board
Parts:
- removed C1, C5: 10u, Capacitor_SMD:C_0805_2012Metric, symbol Device:C
- removed C22: DNF, Capacitor_SMD:C_0402_1005Metric, symbol Device:C
- removed H1, H2, H3, H4: MountingHole, MountingHole:MountingHole_2.7mm_M2.5, symbol Mechanical:MountingHole
- removed J1: USB_B_Micro, Connector_USB:USB_Micro-B_Amphenol_10103594-0001LF_Horizontal, symbol Connector:USB_B_Micro
- removed J2, J3: Conn_02x26_Odd_Even, Connector_PinHeader_2.54mm:PinHeader_2x26_P2.54mm_Vertical, symbol Connector_Generic:Conn_02x26_Odd_Even
- removed J4: SM03B-SRSS-TB, Connector_JST:JST_SH_SM03B-SRSS-TB_1x03-1MP_P1.00mm_Horizontal, symbol Connector_Generic_MountingPin:Conn_01x03_MountingPin
- removed R1, R11, R13, R9: DNF, Resistor_SMD:R_0402_1005Metric, symbol Device:R
- removed R10: 0, Resistor_SMD:R_0402_1005Metric, symbol Device:R
- removed R4, R6: 1k, Resistor_SMD:R_0402_1005Metric, symbol Device:R
- removed SW1, SW2: SW_Push, Button_Switch_SMD:SW_Push_1P1T_NO_Vertical_Wuerth_434133025816, symbol Switch:SW_Push
- removed U2: NCP1117-3.3_SOT223, Package_TO_SOT_SMD:SOT-223-3_TabPin2, symbol Regulator_Linear:NCP1117-3.3_SOT223
- removed U4: DNF, Package_SO:SOIC-8_5.23x5.23mm_P1.27mm, symbol Memory_Flash:W25Q128JVS
- added D1: WS2812B, LED_SMD:LED_WS2812B_PLCC4_5.0x5.0mm_P3.2mm, symbol LED:WS2812B
- added J1, J6: Conn_01x02, Connector_PinHeader_2.00mm:PinHeader_1x02_P2.00mm_Vertical, symbol Connector_Generic:Conn_01x02
- added J2, J3: Conn_01x01, Connector_PinHeader_2.00mm:PinHeader_1x01_P2.00mm_Vertical, symbol Connector_Generic:Conn_01x01
- added J4: Conn_02x10_Odd_Even, Connector_PinHeader_2.00mm:PinHeader_2x10_P2.00mm_Vertical, symbol Connector_Generic:Conn_02x10_Odd_Even
- added J5: Conn_01x04, Connector_PinHeader_2.00mm:PinHeader_1x04_P2.00mm_Vertical, symbol Connector_Generic:Conn_01x04
- added J7: Conn_01x16, Connector_PinHeader_2.00mm:PinHeader_1x16_P2.00mm_Vertical, symbol Connector_Generic:Conn_01x16
- added J9: Conn_01x03, Connector_PinHeader_2.00mm:PinHeader_1x03_P2.00mm_Vertical, symbol Connector_Generic:Conn_01x03
- added JP1: SolderJumper_2_Open, Jumper:SolderJumper-2_P1.3mm_Open_RoundedPad1.0x1.5mm, symbol Jumper:SolderJumper_2_Open
- added U1: IS66WVH8M8ALL-166B1LI, Custom:BGA25C100P5X5_800X600X120N, symbol Custom:IS66WVH8M8ALL-166B1LI
- C14: renamed from C6; footprint RP2350_80QFN_minimal:C_0402_1005Metric_small_pads -> RP2350B_chip_board:C_0402_1005Metric_small_pads
- C15: renamed from C7; footprint RP2350_80QFN_minimal:C_0402_1005Metric_small_pads -> RP2350B_chip_board:C_0402_1005Metric_small_pads
- L1: footprint RP2350_80QFN_minimal:L_pol_2016 -> RP2350B_chip_board:L_pol_2016
- U3: renamed from U1; footprint RP2350_80QFN_minimal:RP2350-QFN-80-1EP_10x10_P0.4mm_EP3.4x3.4mm_ThermalVias -> RP2350B_chip_board:RP2350-QFN-80-1EP_10x10_P0.4mm_EP3.4x3.4mm_ThermalVias
- renumbered C8 to C1, C18 to C10, C20 to C11, C21 to C12, C9 to C13, C2 to C16, C19 to C17, C3 to C18, C4 to C19, C10 to C2, C11 to C3, C12 to C4, C13 to C5, C14 to C6, C15 to C7, C16 to C8, C17 to C9, R3 to R1, R7 to R2, R8 to R3, R2 to R4, U3 to U2
Connections:
- net QSPI_SS is gone; now on net FLASH_SS: U3.75 (QSPI_SS)
- net +3V3: now also D1.1 (VDD), J1.1 (Pin_1), J6.2 (Pin_2)
- net FLASH_SS: now also J3.1 (Pin_1)
- net GND: now also D1.3 (VSS), J5.3 (Pin_3), J6.1 (Pin_1), J9.1 (Pin_1), U1.B3 (VSS), U1.C1 (VSSQ), U1.E5 (VSSQ__1)
- net GPIO0: now also U1.E3 (DQ5)
- net GPIO1: now also U1.C4 (DQ2)
- net GPIO10: now also U1.B1 (~{CK})
- net GPIO11: now also U1.A3 (~{CS})
- net GPIO12: now also J7.16 (Pin_16)
- net GPIO13: now also J7.15 (Pin_15)
- net GPIO14: now also J7.14 (Pin_14)
- net GPIO15: now also J7.13 (Pin_13)
- net GPIO16: now also J7.12 (Pin_12)
- net GPIO17: now also J7.11 (Pin_11)
- net GPIO18: now also J7.10 (Pin_10)
- net GPIO19: now also J7.9 (Pin_9)
- net GPIO2: now also U1.D5 (DQ4)
- net GPIO20: now also J7.8 (Pin_8)
- net GPIO21: now also J7.7 (Pin_7)
- net GPIO22: now also J7.6 (Pin_6)
- net GPIO23: now also J7.5 (Pin_5)
- net GPIO24: now also J7.4 (Pin_4)
- net GPIO25: now also J7.3 (Pin_3)
- net GPIO26: now also J7.2 (Pin_2)
- net GPIO27: now also J7.1 (Pin_1)
- net GPIO28: now also J4.1 (Pin_1)
- net GPIO29: now also J4.2 (Pin_2)
- net GPIO3: now also U1.D4 (DQ3)
- net GPIO30: now also J4.3 (Pin_3)
- net GPIO31: now also J4.4 (Pin_4)
- net GPIO32: now also J4.5 (Pin_5)
- net GPIO33: now also J4.6 (Pin_6)
- net GPIO34: now also J4.7 (Pin_7)
- net GPIO35: now also J4.8 (Pin_8)
- net GPIO36: now also J4.9 (Pin_9)
- net GPIO37: now also J4.10 (Pin_10)
- net GPIO38: now also J4.11 (Pin_11)
- net GPIO39: now also J4.12 (Pin_12)
- net GPIO4: now also U1.D3 (DQ0)
- net GPIO40_ADC0: now also J4.13 (Pin_13)
- net GPIO41_ADC1: now also J4.14 (Pin_14)
- net GPIO42_ADC2: now also J4.15 (Pin_15)
- net GPIO43_ADC3: now also J4.16 (Pin_16)
- net GPIO44_ADC4: now also J4.17 (Pin_17)
- net GPIO45_ADC5: now also J4.18 (Pin_18)
- net GPIO46_ADC6: now also J4.19 (Pin_19)
- net GPIO47_ADC7: now also J4.20 (Pin_20), JP1.1 (A)
- net GPIO5: now also U1.E2 (DQ6)
- net GPIO6: now also U1.D2 (DQ1)
- net GPIO7: now also U1.E1 (DQ7)
- net GPIO8: now also U1.C3 (RWDS)
- net GPIO9: now also U1.B2 (CK)
- net RUN: now also J5.1 (Pin_1)
- net SWCLK: now also J5.4 (Pin_4)
- net SWD: now also J5.2 (Pin_2)
- net USB_D+: now also J9.2 (Pin_2)
- net USB_D-: now also J9.3 (Pin_3)
- new net: J1.2 (Pin_2), U1.B4 (VCC), U1.D1 (VCCQ), U1.E4 (VCCQ__1)
- new net: J2.1 (Pin_1), U1.A4 (~{RESET})
- new net: D1.4 (DIN), JP1.2 (B)
Other:
- note removed: "IOs"
- note removed: "JST Debug Connector"
- note removed: "Optional Secondary flash or PSRAM (U4), using the second chip select (XIP_SS_N[1]) on GPIO0. N.B. Pull-up R13 will be required as GPIOs default to pull-downs at power-up."
- note removed: "Power"
- note removed: "Secondary Flash/PSRAM"
- moved on the sheet: C17
