File: boards/pcie/disp.kicad_sch (KiCad schematic)
At the start: 0 parts

Commit message: pcie: add leds, buck regulators
Parts:
- added C100, C101, C102, C103, C104, C105, C106, C107, C108, C109, C110, C111, C112, C113, C114, C115, C116, C117, C118, C119, C120, C121, C122, C123, C124, C125, C126, C127, C128, C129, C130, C131, C132, C133, C134, C135, C136, C137, C138, C139, C140, C141, C142, C143, C144, C145, C146, C147, C148, C149, C150, C151, C152, C153, C154, C155, C156, C157, C158, C159, C160, C161, C162, C163, C164, C165, C166, C167, C168, C169, C170, C171, C172, C173, C174, C175, C176, C177, C178, C179, C180, C19, C20, C21, C22, C23, C24, C25, C26, C27, C28, C29, C30, C31, C32, C37, C66, C67, C68, C69, C70, C71, C72, C73, C74, C75, C76, C77, C78, C79, C80, C81, C82, C83, C84, C85, C86, C87, C88, C89, C90, C91, C92, C93, C94, C95, C96, C97, C98, C99: 100nF, Capacitor_SMD:C_0402_1005Metric, symbol Device:C
- added D10, D100, D101, D102, D103, D104, D105, D106, D107, D108, D109, D11, D110, D111, D112, D113, D114, D115, D116, D117, D118, D119, D12, D120, D121, D122, D123, D124, D125, D126, D127, D128, D129, D13, D130, D131, D132, D133, D134, D135, D136, D137, D138, D139, D14, D140, D141, D142, D143, D144, D145, D146, D147, D148, D149, D15, D150, D151, D152, D153, D154, D155, D156, D157, D158, D159, D16, D160, D161, D162, D163, D164, D165, D166, D167, D168, D169, D17, D170, D171, D172, D173, D174, D175, D176, D177, D178, D179, D18, D180, D181, D182, D183, D184, D185, D186, D187, D188, D189, D19, D190, D191, D192, D193, D194, D195, D196, D197, D198, D20, D21, D22, D23, D24, D25, D26, D27, D28, D29, D30, D31, D32, D33, D34, D35, D36, D37, D38, D39, D40, D41, D42, D43, D44, D45, D46, D47, D48, D49, D50, D51, D52, D53, D54, D55, D56, D57, D58, D59, D60, D61, D62, D63, D64, D65, D66, D67, D68, D69, D7, D70, D71, D72, D73, D74, D75, D76, D77, D78, D79, D8, D80, D81, D82, D83, D84, D85, D86, D87, D88, D89, D9, D90, D91, D92, D93, D94, D95, D96, D97, D98, D99: LED_45deg, pcie:LED_WS2812B-2020_PLCC4_2.0x2.0mm, symbol LED:WS2812B-2020
Connections:
- new net: D60.1 (DOUT), D61.3 (DIN)
- new net: D59.1 (DOUT), D60.3 (DIN)
- new net: D36.1 (DOUT), D37.3 (DIN)
- new net: D35.1 (DOUT), D36.3 (DIN)
- new net: D45.1 (DOUT), D46.3 (DIN)
- new net: D44.1 (DOUT), D45.3 (DIN)
- new net: D139.1 (DOUT), D140.3 (DIN)
- new net: D138.1 (DOUT), D139.3 (DIN)
- new net: D109.1 (DOUT), D110.3 (DIN)
- new net: D108.1 (DOUT), D109.3 (DIN)
- new net: D177.1 (DOUT), D178.3 (DIN)
- new net: D176.1 (DOUT), D177.3 (DIN)
- new net: D149.1 (DOUT), D150.3 (DIN)
- new net: D148.1 (DOUT), D149.3 (DIN)
- new net: D34.1 (DOUT), D35.3 (DIN)
- new net: D55.1 (DOUT), D56.3 (DIN)
- new net: D54.1 (DOUT), D55.3 (DIN)
- new net: D75.1 (DOUT), D76.3 (DIN)
- new net: D74.1 (DOUT), D75.3 (DIN)
- new net: D105.1 (DOUT), D106.3 (DIN)
- new net: D104.1 (DOUT), D105.3 (DIN)
- new net: D144.1 (DOUT), D145.3 (DIN)
- new net: D143.1 (DOUT), D144.3 (DIN)
- new net: D61.1 (DOUT), D62.3 (DIN)
- new net: D76.1 (DOUT), D77.3 (DIN)
- new net: D173.1 (DOUT), D174.3 (DIN)
- new net: D172.1 (DOUT), D173.3 (DIN)
- new net: D71.1 (DOUT), D72.3 (DIN)
- new net: D70.1 (DOUT), D71.3 (DIN)
- new net: D67.1 (DOUT), D68.3 (DIN)
- new net: D66.1 (DOUT), D67.3 (DIN)
- new net: D171.1 (DOUT), D172.3 (DIN)
- new net: D170.1 (DOUT), D171.3 (DIN)
- new net: D58.1 (DOUT), D59.3 (DIN)
- new net: D57.1 (DOUT), D58.3 (DIN)
- new net: D51.1 (DOUT), D52.3 (DIN)
- new net: D50.1 (DOUT), D51.3 (DIN)
- new net: D52.1 (DOUT), D53.3 (DIN)
- new net: D37.1 (DOUT), D38.3 (DIN)
- new net: D62.1 (DOUT), D63.3 (DIN)
- new net: D43.1 (DOUT), D44.3 (DIN)
- new net: D92.1 (DOUT), D93.3 (DIN)
- new net: D91.1 (DOUT), D92.3 (DIN)
- new net: D87.1 (DOUT), D88.3 (DIN)
- new net: D86.1 (DOUT), D87.3 (DIN)
- new net: D128.1 (DOUT), D129.3 (DIN)
- new net: D127.1 (DOUT), D128.3 (DIN)
- new net: D188.1 (DOUT), D189.3 (DIN)
- new net: D187.1 (DOUT), D188.3 (DIN)
- new net: D146.1 (DOUT), D147.3 (DIN)
- new net: D145.1 (DOUT), D146.3 (DIN)
- new net: D160.1 (DOUT), D161.3 (DIN)
- new net: D159.1 (DOUT), D160.3 (DIN)
- new net: D79.1 (DOUT), D80.3 (DIN)
- new net: D78.1 (DOUT), D79.3 (DIN)
- new net: D142.1 (DOUT), D143.3 (DIN)
- new net: D117.1 (DOUT), D118.3 (DIN)
- new net: D116.1 (DOUT), D117.3 (DIN)
- new net: D93.1 (DOUT), D94.3 (DIN)
- new net: D122.1 (DOUT), D123.3 (DIN)
- new net: D121.1 (DOUT), D122.3 (DIN)
- new net: D119.1 (DOUT), D120.3 (DIN)
- new net: D118.1 (DOUT), D119.3 (DIN)
- new net: D103.1 (DOUT), D104.3 (DIN)
- new net: D102.1 (DOUT), D103.3 (DIN)
- new net: D48.1 (DOUT), D49.3 (DIN)
- new net: D47.1 (DOUT), D48.3 (DIN)
- new net: D32.1 (DOUT), D33.3 (DIN)
- new net: D31.1 (DOUT), D32.3 (DIN)
- new net: D175.1 (DOUT), D176.3 (DIN)
- new net: D174.1 (DOUT), D175.3 (DIN)
- new net: D65.1 (DOUT), D66.3 (DIN)
- new net: D97.1 (DOUT), D98.3 (DIN)
- new net: D96.1 (DOUT), D97.3 (DIN)
- new net: D101.1 (DOUT), D102.3 (DIN)
- new net: D100.1 (DOUT), D101.3 (DIN)
- new net: D26.1 (DOUT), D27.3 (DIN)
- new net: D25.1 (DOUT), D26.3 (DIN)
- new net: D18.1 (DOUT), D19.3 (DIN)
- new net: D17.1 (DOUT), D18.3 (DIN)
- new net: D152.1 (DOUT), D153.3 (DIN)
- new net: D151.1 (DOUT), D152.3 (DIN)
- new net: D123.1 (DOUT), D124.3 (DIN)
- new net: D181.1 (DOUT), D182.3 (DIN)
- new net: D180.1 (DOUT), D181.3 (DIN)
- new net: D94.1 (DOUT), D95.3 (DIN)
- new net: D164.1 (DOUT), D165.3 (DIN)
- new net: D163.1 (DOUT), D164.3 (DIN)
- new net: D166.1 (DOUT), D167.3 (DIN)
- new net: D165.1 (DOUT), D166.3 (DIN)
- new net: D186.1 (DOUT), D187.3 (DIN)
- new net: D185.1 (DOUT), D186.3 (DIN)
- new net: D136.1 (DOUT), D137.3 (DIN)
- new net: D135.1 (DOUT), D136.3 (DIN)
- new net: D192.1 (DOUT), D193.3 (DIN)
- new net: D191.1 (DOUT), D192.3 (DIN)
- new net: D158.1 (DOUT), D159.3 (DIN)
- new net: D157.1 (DOUT), D158.3 (DIN)
- new net: D189.1 (DOUT), D190.3 (DIN)
- new net: D24.1 (DOUT), D25.3 (DIN)
- new net: D23.1 (DOUT), D24.3 (DIN)
- new net: D8.1 (DOUT), D9.3 (DIN)
- new net: D7.1 (DOUT), D8.3 (DIN)
- new net: D29.1 (DOUT), D30.3 (DIN)
- new net: D28.1 (DOUT), D29.3 (DIN)
- new net: D21.1 (DOUT), D22.3 (DIN)
- new net: D20.1 (DOUT), D21.3 (DIN)
- new net: D81.1 (DOUT), D82.3 (DIN)
- new net: D80.1 (DOUT), D81.3 (DIN)
- new net: D193.1 (DOUT), D194.3 (DIN)
- new net: D56.1 (DOUT), D57.3 (DIN)
- new net: D95.1 (DOUT), D96.3 (DIN)
- new net: D16.1 (DOUT), D17.3 (DIN)
- new net: D190.1 (DOUT), D191.3 (DIN)
- new net: D147.1 (DOUT), D148.3 (DIN)
- new net: D39.1 (DOUT), D40.3 (DIN)
- new net: D38.1 (DOUT), D39.3 (DIN)
- new net: D107.1 (DOUT), D108.3 (DIN)
- new net: D161.1 (DOUT), D162.3 (DIN)
- new net: D134.1 (DOUT), D135.3 (DIN)
- new net: D98.1 (DOUT), D99.3 (DIN)
- new net: D19.1 (DOUT), D20.3 (DIN)
- new net: D115.1 (DOUT), D116.3 (DIN)
- new net: D15.1 (DOUT), D16.3 (DIN)
- new net: D14.1 (DOUT), D15.3 (DIN)
- new net: D85.1 (DOUT), D86.3 (DIN)
- new net: D106.1 (DOUT), D107.3 (DIN)
- new net: D53.1 (DOUT), D54.3 (DIN)
- new net: D162.1 (DOUT), D163.3 (DIN)
- new net: D154.1 (DOUT), D155.3 (DIN)
- new net: D153.1 (DOUT), D154.3 (DIN)
- new net: D42.1 (DOUT), D43.3 (DIN)
- new net: D41.1 (DOUT), D42.3 (DIN)
- new net: D132.1 (DOUT), D133.3 (DIN)
- new net: D131.1 (DOUT), D132.3 (DIN)
- new net: D168.1 (DOUT), D169.3 (DIN)
- new net: D167.1 (DOUT), D168.3 (DIN)
- new net: D197.1 (DOUT), D198.3 (DIN)
- new net: D178.1 (DOUT), D179.3 (DIN)
- new net: D33.1 (DOUT), D34.3 (DIN)
- new net: D13.1 (DOUT), D14.3 (DIN)
- new net: D72.1 (DOUT), D73.3 (DIN)
- new net: D141.1 (DOUT), D142.3 (DIN)
- new net: D140.1 (DOUT), D141.3 (DIN)
- new net: D196.1 (DOUT), D197.3 (DIN)
- new net: D195.1 (DOUT), D196.3 (DIN)
- new net: D130.1 (DOUT), D131.3 (DIN)
- new net: D129.1 (DOUT), D130.3 (DIN)
- new net: D12.1 (DOUT), D13.3 (DIN)
- new net: D77.1 (DOUT), D78.3 (DIN)
- new net: D137.1 (DOUT), D138.3 (DIN)
- new net: D194.1 (DOUT), D195.3 (DIN)
- new net: D114.1 (DOUT), D115.3 (DIN)
- new net: D113.1 (DOUT), D114.3 (DIN)
- new net: D156.1 (DOUT), D157.3 (DIN)
- new net: D155.1 (DOUT), D156.3 (DIN)
- new net: D179.1 (DOUT), D180.3 (DIN)
- new net: D111.1 (DOUT), D112.3 (DIN)
- new net: D110.1 (DOUT), D111.3 (DIN)
- new net: D100.3 (DIN), D99.1 (DOUT)
- new net: D90.1 (DOUT), D91.3 (DIN)
- new net: D89.1 (DOUT), D90.3 (DIN)
- new net: D68.1 (DOUT), D69.3 (DIN)
- new net: D126.1 (DOUT), D127.3 (DIN)
- new net: D30.1 (DOUT), D31.3 (DIN)
- new net: D84.1 (DOUT), D85.3 (DIN)
- new net: D184.1 (DOUT), D185.3 (DIN)
- new net: D10.3 (DIN), D9.1 (DOUT)
- new net: D150.1 (DOUT), D151.3 (DIN)
- new net: D64.1 (DOUT), D65.3 (DIN)
- new net: D63.1 (DOUT), D64.3 (DIN)
- new net: D82.1 (DOUT), D83.3 (DIN)
- new net: D73.1 (DOUT), D74.3 (DIN)
- new net: D133.1 (DOUT), D134.3 (DIN)
- new net: D22.1 (DOUT), D23.3 (DIN)
- new net: D40.1 (DOUT), D41.3 (DIN)
- new net: D169.1 (DOUT), D170.3 (DIN)
- new net: D88.1 (DOUT), D89.3 (DIN)
- new net: D46.1 (DOUT), D47.3 (DIN)
- new net: D182.1 (DOUT), D183.3 (DIN)
- new net: D27.1 (DOUT), D28.3 (DIN)
- new net: D124.1 (DOUT), D125.3 (DIN)
- new net: D69.1 (DOUT), D70.3 (DIN)
- new net: D49.1 (DOUT), D50.3 (DIN)
- new net: D83.1 (DOUT), D84.3 (DIN)
- new net: D125.1 (DOUT), D126.3 (DIN)
- new net: D112.1 (DOUT), D113.3 (DIN)
- new net: D11.1 (DOUT), D12.3 (DIN)
- new net: D10.1 (DOUT), D11.3 (DIN)
- new net: D120.1 (DOUT), D121.3 (DIN)
- new net: D183.1 (DOUT), D184.3 (DIN)
- new net GND: C100.2, C101.2, C102.2, C103.2, C104.2, C105.2, C106.2, C107.2, C108.2, C109.2, C110.2, C111.2, C112.2, C113.2, C114.2, C115.2, C116.2, C117.2, C118.2, C119.2, C120.2, C121.2, C122.2, C123.2, C124.2, C125.2, C126.2, C127.2, C128.2, C129.2, C130.2, C131.2, C132.2, C133.2, C134.2, C135.2, C136.2, C137.2, C138.2, C139.2, C140.2, C141.2, C142.2, C143.2, C144.2, C145.2, C146.2, C147.2, C148.2, C149.2, C150.2, C151.2, C152.2, C153.2, C154.2, C155.2, C156.2, C157.2, C158.2, C159.2, C160.2, C161.2, C162.2, C163.2, C164.2, C165.2, C166.2, C167.2, C168.2, C169.2, C170.2, C171.2, C172.2, C173.2, C174.2, C175.2, C176.2, C177.2, C178.2, C179.2, C180.2, C19.2, C20.2, C21.2, C22.2, C23.2, C24.2, C25.2, C26.2, C27.2, C28.2, C29.2, C30.2, C31.2, C32.2, C37.2, C66.2, C67.2, C68.2, C69.2, C70.2, C71.2, C72.2, C73.2, C74.2, C75.2, C76.2, C77.2, C78.2, C79.2, C80.2, C81.2, C82.2, C83.2, C84.2, C85.2, C86.2, C87.2, C88.2, C89.2, C90.2, C91.2, C92.2, C93.2, C94.2, C95.2, C96.2, C97.2, C98.2, C99.2, D10.2 (VSS), D100.2 (VSS), D101.2 (VSS), D102.2 (VSS), D103.2 (VSS), D104.2 (VSS), D105.2 (VSS), D106.2 (VSS), D107.2 (VSS), D108.2 (VSS), D109.2 (VSS), D11.2 (VSS), D110.2 (VSS), D111.2 (VSS), D112.2 (VSS), D113.2 (VSS), D114.2 (VSS), D115.2 (VSS), D116.2 (VSS), D117.2 (VSS), D118.2 (VSS), D119.2 (VSS), D12.2 (VSS), D120.2 (VSS), D121.2 (VSS), D122.2 (VSS), D123.2 (VSS), D124.2 (VSS), D125.2 (VSS), D126.2 (VSS), D127.2 (VSS), D128.2 (VSS), D129.2 (VSS), D13.2 (VSS), D130.2 (VSS), D131.2 (VSS), D132.2 (VSS), D133.2 (VSS), D134.2 (VSS), D135.2 (VSS), D136.2 (VSS), D137.2 (VSS), D138.2 (VSS), D139.2 (VSS), D14.2 (VSS), D140.2 (VSS), D141.2 (VSS), D142.2 (VSS), D143.2 (VSS), D144.2 (VSS), D145.2 (VSS), D146.2 (VSS), D147.2 (VSS), D148.2 (VSS), D149.2 (VSS), D15.2 (VSS), D150.2 (VSS), D151.2 (VSS), D152.2 (VSS), D153.2 (VSS), D154.2 (VSS), D155.2 (VSS), D156.2 (VSS), D157.2 (VSS), D158.2 (VSS), D159.2 (VSS), D16.2 (VSS), D160.2 (VSS), D161.2 (VSS), D162.2 (VSS), D163.2 (VSS), D164.2 (VSS), D165.2 (VSS), D166.2 (VSS), D167.2 (VSS), D168.2 (VSS), D169.2 (VSS), D17.2 (VSS), D170.2 (VSS), D171.2 (VSS), D172.2 (VSS), D173.2 (VSS), D174.2 (VSS), D175.2 (VSS), D176.2 (VSS), D177.2 (VSS), D178.2 (VSS), D179.2 (VSS), D18.2 (VSS), D180.2 (VSS), D181.2 (VSS), D182.2 (VSS), D183.2 (VSS), D184.2 (VSS), D185.2 (VSS), D186.2 (VSS), D187.2 (VSS), D188.2 (VSS), D189.2 (VSS), D19.2 (VSS), D190.2 (VSS), D191.2 (VSS), D192.2 (VSS), D193.2 (VSS), D194.2 (VSS), D195.2 (VSS), D196.2 (VSS), D197.2 (VSS), D198.2 (VSS), D20.2 (VSS), D21.2 (VSS), D22.2 (VSS), D23.2 (VSS), D24.2 (VSS), D25.2 (VSS), D26.2 (VSS), D27.2 (VSS), D28.2 (VSS), D29.2 (VSS), D30.2 (VSS), D31.2 (VSS), D32.2 (VSS), D33.2 (VSS), D34.2 (VSS), D35.2 (VSS), D36.2 (VSS), D37.2 (VSS), D38.2 (VSS), D39.2 (VSS), D40.2 (VSS), D41.2 (VSS), D42.2 (VSS), D43.2 (VSS), D44.2 (VSS), D45.2 (VSS), D46.2 (VSS), D47.2 (VSS), D48.2 (VSS), D49.2 (VSS), D50.2 (VSS), D51.2 (VSS), D52.2 (VSS), D53.2 (VSS), D54.2 (VSS), D55.2 (VSS), D56.2 (VSS), D57.2 (VSS), D58.2 (VSS), D59.2 (VSS), D60.2 (VSS), D61.2 (VSS), D62.2 (VSS), D63.2 (VSS), D64.2 (VSS), D65.2 (VSS), D66.2 (VSS), D67.2 (VSS), D68.2 (VSS), D69.2 (VSS), D7.2 (VSS), D70.2 (VSS), D71.2 (VSS), D72.2 (VSS), D73.2 (VSS), D74.2 (VSS), D75.2 (VSS), D76.2 (VSS), D77.2 (VSS), D78.2 (VSS), D79.2 (VSS), D8.2 (VSS), D80.2 (VSS), D81.2 (VSS), D82.2 (VSS), D83.2 (VSS), D84.2 (VSS), D85.2 (VSS), D86.2 (VSS), D87.2 (VSS), D88.2 (VSS), D89.2 (VSS), D9.2 (VSS), D90.2 (VSS), D91.2 (VSS), D92.2 (VSS), D93.2 (VSS), D94.2 (VSS), D95.2 (VSS), D96.2 (VSS), D97.2 (VSS), D98.2 (VSS), D99.2 (VSS)
- new net LED_5V1: C149.1, C150.1, C151.1, C152.1, C153.1, C154.1, C155.1, C156.1, C157.1, C158.1, C159.1, C160.1, C161.1, C162.1, C163.1, C164.1, C165.1, C166.1, C167.1, C168.1, C169.1, C170.1, C171.1, C172.1, C173.1, C174.1, C175.1, C176.1, C177.1, C178.1, C179.1, C180.1, C19.1, C20.1, C21.1, C22.1, C27.1, C28.1, C29.1, C30.1, C31.1, C32.1, C37.1, C66.1, C67.1, C68.1, C69.1, C70.1, C71.1, C72.1, C73.1, C74.1, C75.1, C76.1, C77.1, C78.1, C79.1, C80.1, C81.1, C82.1, C83.1, C84.1, C85.1, C86.1, C87.1, D10.4 (VDD), D100.4 (VDD), D101.4 (VDD), D102.4 (VDD), D11.4 (VDD), D12.4 (VDD), D13.4 (VDD), D14.4 (VDD), D15.4 (VDD), D16.4 (VDD), D17.4 (VDD), D18.4 (VDD), D19.4 (VDD), D20.4 (VDD), D21.4 (VDD), D22.4 (VDD), D23.4 (VDD), D24.4 (VDD), D25.4 (VDD), D26.4 (VDD), D27.4 (VDD), D28.4 (VDD), D29.4 (VDD), D30.4 (VDD), D31.4 (VDD), D32.4 (VDD), D33.4 (VDD), D34.4 (VDD), D35.4 (VDD), D36.4 (VDD), D37.4 (VDD), D38.4 (VDD), D39.4 (VDD), D40.4 (VDD), D41.4 (VDD), D42.4 (VDD), D43.4 (VDD), D44.4 (VDD), D45.4 (VDD), D46.4 (VDD), D47.4 (VDD), D48.4 (VDD), D49.4 (VDD), D50.4 (VDD), D51.4 (VDD), D52.4 (VDD), D53.4 (VDD), D54.4 (VDD), D55.4 (VDD), D56.4 (VDD), D57.4 (VDD), D58.4 (VDD), D59.4 (VDD), D60.4 (VDD), D61.4 (VDD), D62.4 (VDD), D63.4 (VDD), D64.4 (VDD), D65.4 (VDD), D66.4 (VDD), D67.4 (VDD), D68.4 (VDD), D69.4 (VDD), D7.4 (VDD), D70.4 (VDD), D71.4 (VDD), D72.4 (VDD), D73.4 (VDD), D74.4 (VDD), D75.4 (VDD), D76.4 (VDD), D77.4 (VDD), D78.4 (VDD), D79.4 (VDD), D8.4 (VDD), D80.4 (VDD), D81.4 (VDD), D82.4 (VDD), D83.4 (VDD), D84.4 (VDD), D85.4 (VDD), D86.4 (VDD), D87.4 (VDD), D88.4 (VDD), D89.4 (VDD), D9.4 (VDD), D90.4 (VDD), D91.4 (VDD), D92.4 (VDD), D93.4 (VDD), D94.4 (VDD), D95.4 (VDD), D96.4 (VDD), D97.4 (VDD), D98.4 (VDD), D99.4 (VDD)
- new net LED_5V2: C100.1, C101.1, C102.1, C103.1, C104.1, C105.1, C106.1, C107.1, C108.1, C109.1, C110.1, C111.1, C112.1, C113.1, C114.1, C115.1, C116.1, C117.1, C118.1, C119.1, C120.1, C121.1, C122.1, C123.1, C124.1, C125.1, C126.1, C127.1, C128.1, C129.1, C130.1, C131.1, C132.1, C133.1, C134.1, C135.1, C136.1, C137.1, C138.1, C139.1, C140.1, C141.1, C142.1, C143.1, C144.1, C145.1, C146.1, C147.1, C148.1, C23.1, C24.1, C25.1, C26.1, C88.1, C89.1, C90.1, C91.1, C92.1, C93.1, C94.1, C95.1, C96.1, C97.1, C98.1, C99.1, D103.4 (VDD), D104.4 (VDD), D105.4 (VDD), D106.4 (VDD), D107.4 (VDD), D108.4 (VDD), D109.4 (VDD), D110.4 (VDD), D111.4 (VDD), D112.4 (VDD), D113.4 (VDD), D114.4 (VDD), D115.4 (VDD), D116.4 (VDD), D117.4 (VDD), D118.4 (VDD), D119.4 (VDD), D120.4 (VDD), D121.4 (VDD), D122.4 (VDD), D123.4 (VDD), D124.4 (VDD), D125.4 (VDD), D126.4 (VDD), D127.4 (VDD), D128.4 (VDD), D129.4 (VDD), D130.4 (VDD), D131.4 (VDD), D132.4 (VDD), D133.4 (VDD), D134.4 (VDD), D135.4 (VDD), D136.4 (VDD), D137.4 (VDD), D138.4 (VDD), D139.4 (VDD), D140.4 (VDD), D141.4 (VDD), D142.4 (VDD), D143.4 (VDD), D144.4 (VDD), D145.4 (VDD), D146.4 (VDD), D147.4 (VDD), D148.4 (VDD), D149.4 (VDD), D150.4 (VDD), D151.4 (VDD), D152.4 (VDD), D153.4 (VDD), D154.4 (VDD), D155.4 (VDD), D156.4 (VDD), D157.4 (VDD), D158.4 (VDD), D159.4 (VDD), D160.4 (VDD), D161.4 (VDD), D162.4 (VDD), D163.4 (VDD), D164.4 (VDD), D165.4 (VDD), D166.4 (VDD), D167.4 (VDD), D168.4 (VDD), D169.4 (VDD), D170.4 (VDD), D171.4 (VDD), D172.4 (VDD), D173.4 (VDD), D174.4 (VDD), D175.4 (VDD), D176.4 (VDD), D177.4 (VDD), D178.4 (VDD), D179.4 (VDD), D180.4 (VDD), D181.4 (VDD), D182.4 (VDD), D183.4 (VDD), D184.4 (VDD), D185.4 (VDD), D186.4 (VDD), D187.4 (VDD), D188.4 (VDD), D189.4 (VDD), D190.4 (VDD), D191.4 (VDD), D192.4 (VDD), D193.4 (VDD), D194.4 (VDD), D195.4 (VDD), D196.4 (VDD), D197.4 (VDD), D198.4 (VDD)
- no-connect marks 0 -> 1
