File: boards/pcie/pcie.kicad_sch (KiCad schematic)
At the start: 2 parts, among them J1 PCIexpress_bracket, J2 PCIexpress_x16

Commit message: pcie: add leds, buck regulators
Parts:
- added H1, H2: MountingHole, MountingHole:MountingHole_3.2mm_M3_Pad, symbol Mechanical:MountingHole
- added J12: Conn_02x03_Odd_Even, Connector_Molex:Molex_Mini-Fit_Jr_5569-06A1_2x03_P4.20mm_Horizontal, symbol Connector_Generic:Conn_02x03_Counter_Clockwise
Connections:
- net GND: now also J12.4 (Pin_4), J12.6 (Pin_6)
- new net +12VE: J12.1 (Pin_1), J12.3 (Pin_3)
- no-connect marks 67 -> 69
