File: boards/pcie/psus.kicad_sch (KiCad schematic)
At the start: 22 parts, among them U1 AP63203WU, U3 AP63205WU, U4 TLV75801PDBVR

Commit message: pcie: add leds, buck regulators
Parts:
- added C181, C187: 22uF@25V, Capacitor_SMD:C_1210_3225Metric, symbol Device:C
- added C182, C186: 220uF@25V, Capacitor_SMD:CP_Elec_6.3x7.7, symbol Device:C_Polarized_US
- added C183, C191: 470uF@16V, Capacitor_SMD:CP_Elec_8x10.5, symbol Device:C_Polarized_US
- added C184, C190: 22uF@10V, Capacitor_SMD:C_1206_3216Metric, symbol Device:C
- added C185, C189: 33nF, Capacitor_SMD:C_0402_1005Metric, symbol Device:C
- added C188, C65: 1uF, Capacitor_SMD:C_0603_1608Metric, symbol Device:C
- added D199, D200: SS1045-SMB, Diode_SMD:D_SMB, symbol Device:D
- added L5, L6: 33uH, Inductor_SMD:L_APV_APH1050, symbol Device:L
- added R53, R55: 3k, Resistor_SMD:R_0402_1005Metric, symbol Device:R
- added R54, R56: 1k, Resistor_SMD:R_0402_1005Metric, symbol Device:R
- added U10, U9: XL4015, Package_TO_SOT_SMD:TO-263-5_TabPin3, symbol Regulator_Switching:XL4015
- C39, C41: value 100n -> 100nF
- C42, C46, C50, C51, C52: value 10u -> 10uF
- C43, C44, C45, C47, C48, C49, C53: value 22u -> 22uF
Connections:
- net GND: now also C181.2, C182.2, C183.2, C184.2, C185.2, C186.2, C187.2, C189.2, C190.2, C191.2, D199.2 (A), D200.2 (A), R54.2, R56.2, U10.1 (GND), U9.1 (GND)
- new net: C188.2, U10.4 (VC)
- new net: C189.1, R55.2, R56.1, U10.2 (FB)
- new net: D200.1 (K), L6.1, U10.3 (SW)
- new net: C65.2, U9.4 (VC)
- new net: C185.1, R53.2, R54.1, U9.2 (FB)
- new net: D199.1 (K), L5.1, U9.3 (SW)
- new net +12VE: C181.1, C182.1, C186.1, C187.1, C188.1, C65.1, U10.5 (VIN), U9.5 (VIN)
- new net LED_5V1: C190.1, C191.1, L6.2, R55.1
- new net LED_5V2: C183.1, C184.1, L5.2, R53.1
