File: boards/pcie/usb-hubs.kicad_sch (KiCad schematic)
At the start: 32 parts, among them U5 CH334F, U6 CH334F, U7 CH334F, U8 CH334F

Commit message: pcie: add leds, buck regulators
Parts:
- C10, C11, C14, C15, C18, C3, C5, C7: value 1u -> 1uF
- C12, C13, C16, C17, C4, C6, C8, C9: value 100n -> 100nF
Changed lines of the file:
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@@
 			)
 		)
-		(property "Value" "100n"
+		(property "Value" "100nF"
 			(at 80.264 45.212 0)
 			(show_name no)
@@
 			)
 		)
-		(property "Value" "1u"
+		(property "Value" "1uF"
 			(at 105.156 132.842 0)
 			(show_name no)
@@
 			)
 		)
-		(property "Value" "100n"
+		(property "Value" "100nF"
 			(at 160.274 49.022 0)
 			(show_name no)
@@
 			)
 		)
-		(property "Value" "100n"
+		(property "Value" "100nF"
 			(at 172.466 132.842 0)
 			(show_name no)
@@
 			)
 		)
-		(property "Value" "1u"
+		(property "Value" "1uF"
 			(at 105.156 45.212 0)
 			(show_name no)
@@
 			)
 		)
-		(property "Value" "1u"
+		(property "Value" "1uF"
 			(at 75.184 45.212 0)
 			(show_name no)
@@
 			)
 		)
-		(property "Value" "1u"
+		(property "Value" "1uF"
 			(at 185.166 49.022 0)
 			(show_name no)
@@
 			)
 		)
-		(property "Value" "1u"
+		(property "Value" "1uF"
 			(at 155.194 49.022 0)
 			(show_name no)
@@
 			)
 		)
-		(property "Value" "1u"
+		(property "Value" "1uF"
 			(at 147.574 132.842 0)
 			(show_name no)
@@
 			)
 		)
-		(property "Value" "1u"
+		(property "Value" "1uF"
 			(at 75.184 132.842 0)
 			(show_name no)
@@
 			)
 		)
-		(property "Value" "1u"
+		(property "Value" "1uF"
 			(at 177.546 132.842 0)
 			(show_name no)
@@
 			)
 		)
-		(property "Value" "100n"
+		(property "Value" "100nF"
 			(at 100.076 132.842 0)
 			(show_name no)
@@
 			)
 		)
-		(property "Value" "100n"
+		(property "Value" "100nF"
 			(at 100.076 45.212 0)
 			(show_name no)
@@
 			)
 		)
-		(property "Value" "100n"
+		(property "Value" "100nF"
 			(at 80.264 132.842 0)
 			(show_name no)
@@
 			)
 		)
-		(property "Value" "100n"
+		(property "Value" "100nF"
 			(at 152.654 132.842 0)
 			(show_name no)
@@
 			)
 		)
-		(property "Value" "100n"
+		(property "Value" "100nF"
 			(at 180.086 49.022 0)
 			(show_name no)
